File: pcb-coil.kicad_pcb (KiCad board)
At the start: 2 copper layers, 100 x 100 mm, 1 part, among them J1 Conn_01x03_Pin

Commit message: Finish to get manufactured
Parts:
- removed J1: Conn_01x03_Pin, Connector_PinHeader_2.54mm:PinHeader_1x03_P2.54mm_Vertical
- added ?: , , F.Cu at (78.2, 75.5)
- added ?: , , F.Cu at (78.5, 44.2)
- added ?: , , F.Cu at (87.5, 36.5)
- added ?: , , F.Cu at (87.2, 83.5)
- added ?: , , F.Cu at (81.0, 38.5)
- added ?: , , F.Cu at (73.2, 62.2)
- added ?: , , F.Cu at (73.0, 50.0)
- added ?: , , F.Cu at (81.0, 81.5)
- added ?: , , F.Cu at (73.2, 57.8)
- added ?: , , F.Cu at (73.0, 70.0)
- added G1: LOGO, LOGO, B.Cu at (100.0, 60.0)
Routing:
- net /A: track 6063.5 -> 0.00 mm, vias 18 -> 0
- net C: vias 0 -> 9
- net B: vias 0 -> 9
- net A: vias 0 -> 6
- added copper zone on B.Cu, net GND
- added copper zone on In4.Cu, net GND
Other:
- board size 100 x 100 mm -> 32.4 x 51 mm
- copper layers 2 -> 6
- board text added: "A"
- board text added: "B"
- board text added: "C"
- board text added: "SH"
